File: niclas-alarmmelder-pro/niclas-alarmmelder-pro.kicad_pcb (KiCad board)
At the start: 2 copper layers, 107.2 x 33 mm, 23 parts, among them J1 DIN-5_180degree, SW1 SW_SPST, U1 MOUDLE-SEEEDUINO-XIAO-ESP32C3, U2 TME-0503S

Commit message: release ready
Sollte so funktionieren, eine Schraube mag oder mag nicht accessible sein je nach Schalter aber idc worst case reichen auch 2
Parts:
- added GPIO3: TestPoint_THTPad_1.0x1.0mm_Drill0.5mm, TestPoint:TestPoint_THTPad_1.0x1.0mm_Drill0.5mm, F.Cu at (111.5, 48.8)
- added GPOI2: TestPoint_THTPad_1.0x1.0mm_Drill0.5mm, TestPoint:TestPoint_THTPad_1.0x1.0mm_Drill0.5mm, F.Cu at (111.5, 46.2)
- added JP1: SolderJumper_3_Open, Jumper:SolderJumper-3_P1.3mm_Open_RoundedPad1.0x1.5mm_NumberLabels, F.Cu at (122.2, 68.3)
- JP OPT: renamed from OPT
- moved R4 4.74 mm to (115.3, 69.6), turned to -90 degrees
- moved R2 1.44 mm to (101.1, 66.3), turned to 0 degrees
- moved R1 1.44 mm to (95.5, 66.3), turned to 0 degrees
- moved R3 1.41 mm to (106.7, 66.3), turned to 0 degrees
Connections:
- net Net-(U1-PB09_A7_D7_RX) renamed Relaiskontakt
- R4 pad 2: +3V3 -> Net-(JP1-C)
- R420 pad 1: (no net) -> GND
- R420 pad 2: (no net) -> GND
- U1 pad 7: unconnected-(U1-PB08_A6_D6_TX-Pad7) -> Net-(JP1-A)
Routing:
- net Net-(JP1-A): track 0.00 -> 13.4 mm
- net Net-(JP1-C): track 0.00 -> 8.40 mm
- net unconnected-(U1-PA4_A1_D1-Pad2): track 0.00 -> 6.10 mm
- net unconnected-(U1-PA02_A0_D0-Pad1): track 0.00 -> 5.84 mm
- net unconnected-(U1-PA6_A10_D10_MOSI-Pad11): track 24.4 -> 21.9 mm
- net +3V3: track 30.0 -> 28.0 mm
- net Net-(D2-A): track 11.4 -> 9.67 mm
- net Net-(D1-A): track 11.4 -> 9.67 mm
- net Net-(D3-A): track 11.4 -> 9.68 mm
- net unconnected-(U1-PA5_A9_D9_MISO-Pad10): track 20.0 -> 18.3 mm
- net Net-(SW1-B): track 46.6 -> 45.2 mm
- net Net-(U1-PA9_A5_D5_SCL): track 12.7 -> 13.8 mm
- net Net-(U1-PA8_A4_D4_SDA): track 20.4 -> 21.4 mm
- net unconnected-(U1-PA7_A8_D8_SCK-Pad9): track 15.4 -> 14.7 mm
Other:
- outline, holes or cut-outs redrawn
- board text added: "30R WHITE 500R GREEN ULP"
- board text added: "GND Basestation"
- board text added: "My Sleep Schedule Was Severely Harmed in the Making of This Project"
- board text added: "if no dcdc"
- board text added: "pub enum Instruction { Mov(Vector), Pos(Point), Arc(Vector, Vector, ArcDirection), Rep(usize, Vector, Instruction), Pen(i5), Err(ParseError), }.unwrap();;"
- board text added: "v1 2025 Design by FS"
- board text removed: "(c) 2025 Vapianovich B Scharf"
- board text removed: "GND Melder"
- board text removed: "pub enum Instruction { Mov(Vector), Pos(Point), Arc(Vector, Vector, ArcDirection), Rep(usize, Vector, Instruction), Pen(is), Err(ParseError), }.unwrap();;"

Commit message: v1.1
small fixes nothing to worry about :)
Parts:
- moved R420 16.6 mm to (155.0, 47.0)
- moved J1 4.83 mm to (165.6, 58.2)
Routing:
- net Relaiskontakt: track 72.1 -> 68.6 mm
Other:
- outline, holes or cut-outs redrawn
- board text added: "v1.01 2025 Design by FS"
- board text removed: "if no dcdc"
- board text removed: "v1 2025 Design by FS"
Changed lines of the file:
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@@
 				(font
 					(size 1 1)
-					(thickness 0.2)
-					(bold yes)
+					(thickness 0.15)
 				)
 			)
@@
 			)
 			(layer "F.SilkS")
-			(net 12)
 		)
 		(fp_line
@@
 			)
 			(layer "F.SilkS")
-			(net 12)
 		)
 		(fp_line
@@
 			)
 			(layer "F.SilkS")
-			(net 12)
 		)
 		(fp_line
@@
 	(footprint "Connector:5pin din"
 		(layer "F.Cu")
-		(at 165.608 53.34)
+		(at 165.608 58.166)
 		(property "Reference" "J1"
-			(at -3.81 0 0)
+			(at 3.81 -1.524 0)
 			(unlocked yes)
 			(layer "F.SilkS")
+			(hide yes)
 			(effects
 				(font
@@
 		(tags "resistor handsolder")
 		(property "Reference" "R3"
-			(at 0 -1.65 360)
+			(at 0 -1.65 0)
 			(layer "F.SilkS")
 			(effects
@@
 		)
 		(property "Value" "R"
-			(at 0 1.65 360)
+			(at 0 1.65 0)
 			(layer "F.Fab")
 			(effects
@@
 		)
 		(fp_text user "${REFERENCE}"
-			(at 0 0 360)
+			(at 0 0 0)
 			(layer "F.Fab")
 			(effects
@@
 				(font
 					(size 1 1)
-					(thickness 0.2)
-					(bold yes)
+					(thickness 0.15)
 				)
 			)
@@
 	(footprint "Resistor_SMD:R_0805_2012Metric"
 		(layer "F.Cu")
-		(at 151.892 63.246)
+		(at 155.0435 46.99)
 		(descr "Resistor SMD 0805 (2012 Metric), square (rectangular) end terminal, IPC_7351 nominal, (Body size source: IPC-SM-782 page 72, https://www.pcb-3d.com/wordpress/wp-content/uploads/ipc-sm-782a_amendment_1_and_2.pdf), generated with kicad-footprint-generator")
 		(tags "resistor")
@@
 		(layer "B.SilkS")
 	)
-	(gr_line
-		(start 142.24 50.8)
-		(end 147.32 50.8)
-		(stroke
-			(width 0.1)
-			(type default)
-		)
-		(layer "F.SilkS")
-	)
-	(gr_line
-		(start 147.32 50.8)
-		(end 147.32 50.038)
-		(stroke
-			(width 0.1)
-			(type default)
-		)
-		(layer "F.SilkS")
-	)
-	(gr_line
-		(start 147.32 50.038)
-		(end 147.32 50.8)
-		(stroke
-			(width 0.1)
-			(type default)
-		)
-		(layer "F.SilkS")
-	)
-	(gr_line
-		(start 142.24 50.038)
-		(end 142.24 50.8)
-		(stroke
-			(width 0.1)
-			(type default)
-		)
-		(layer "F.SilkS")
-	)
 	(gr_circle
 		(center 80.01 46.99)
@@
 	)
 	(gr_circle
-		(center 172.212 48.006)
-		(end 173.228 49.276)
+		(center 172.212 46.99)
+		(end 173.228 48.26)
 		(stroke
 			(width 0.05)
@@
 		)
 	)
-	(gr_text "v1 2025\nDesign by FS"
-		(at 167.132 73.406 0)
+	(gr_text "v1.01 2025\nDesign by FS"
+		(at 168.402 74.168 0)
 		(layer "F.Cu" knockout)
 		(effects
@@
 			(font
 				(size 1 1)
-				(thickness 0.2)
-				(bold yes)
+				(thickness 0.15)
 			)
 			(justify left bottom)
@@
 			(font
 				(size 1 1)
-				(thickness 0.2)
-				(bold yes)
+				(thickness 0.15)
 			)
 			(justify left bottom)
@@
 	)
 	(gr_text "sample text"
-		(at 128.778 70.866 0)
+		(at 128.524 72.898 0)
 		(layer "F.SilkS")
 		(effects
 			(font
 				(size 1 1)
-				(thickness 0.2)
-				(bold yes)
+				(thickness 0.15)
 			)
 			(justify left bottom)
@@
 			(font
 				(size 1 1)
-				(thickness 0.2)
-				(bold yes)
+				(thickness 0.15)
 			)
 			(justify left bottom)
@@
 	)
 	(gr_text "GND Basestation"
-		(at 164.846 53.848 0)
+		(at 158.242 59.436 0)
 		(layer "F.SilkS")
 		(effects
 			(font
 				(size 1 1)
-				(thickness 0.2)
-				(bold yes)
+				(thickness 0.15)
 			)
 			(justify left bottom)
@@
 	)
 	(gr_text "GND"
-		(at 167.132 61.468 0)
-		(layer "F.SilkS")
-		(effects
-			(font
-				(size 1 1)
-				(thickness 0.2)
-				(bold yes)
-			)
-			(justify left bottom)
-		)
-	)
-	(gr_text "if no dcdc"
-		(at 140.208 52.324 0)
+		(at 165.354 67.056 0)
 		(layer "F.SilkS")
 		(effects
 			(font
 				(size 1 1)
-				(thickness 0.1)
+				(thickness 0.15)
 			)
 			(justify left bottom)
@@
 	)
 	(gr_text "BLUNT\nRESISTOR\n"
-		(at 153.924 63.754 0)
+		(at 157.226 47.498 0)
 		(layer "F.SilkS")
 		(effects
 			(font
 				(size 1 1)
-				(thickness 0.2)
-				(bold yes)
+				(thickness 0.15)
 			)
 			(justify left bottom)
@@
 	)
 	(gr_text "NC"
-		(at 166.116 50.038 0)
+		(at 159.766 55.372 0)
 		(layer "F.SilkS")
 		(effects
 			(font
 				(size 1 1)
-				(thickness 0.2)
-				(bold yes)
+				(thickness 0.15)
 			)
 			(justify left bottom)
@@
 	)
 	(gr_text "5V IN"
-		(at 166.116 57.15 0)
+		(at 159.766 63.5 0)
 		(layer "F.SilkS")
 		(effects
 			(font
 				(size 1 1)
-				(thickness 0.2)
-				(bold yes)
+				(thickness 0.15)
 			)
 			(justify left bottom)
@@
 	)
 	(gr_text "to GPIO20"
-		(at 166.878 46.228 0)
+		(at 165.354 51.816 0)
 		(layer "F.SilkS")
 		(effects
 			(font
 				(size 1 1)
-				(thickness 0.2)
-				(bold yes)
+				(thickness 0.15)
 			)
 			(justify left bottom)
@@
 			(font
 				(size 1 1)
-				(thickness 0.2)
-				(bold yes)
+				(thickness 0.15)
 			)
 			(justify left bottom)
@@
 			(font
 				(size 1 1)
-				(thickness 0.2)
-				(bold yes)
+				(thickness 0.15)
 			)
 			(justify left bottom)
@@
 	)
 	(segment
-		(start 136.398 61.468)
-		(end 139.7 64.77)
+		(start 166.116 68.58)
+		(end 167.64 67.056)
 		(width 0.508)
 		(layer "F.Cu")
@@
 	)
 	(segment
-		(start 133.767 61.468)
-		(end 136.398 61.468)
+		(start 149.86 72.898)
+		(end 149.86 70.104)
 		(width 0.508)
 		(layer "F.Cu")
@@
 	)
 	(segment
-		(start 163.83 66.04)
-		(end 167.64 62.23)
+		(start 136.398 61.468)
+		(end 139.7 64.77)
 		(width 0.508)
 		(layer "F.Cu")
@@
 	)
 	(segment
-		(start 149.86 72.898)
-		(end 149.86 67.31)
+		(start 166.116 50.546)
+		(end 162.746 50.546)
 		(width 0.508)
 		(layer "F.Cu")
@@
 	)
 	(segment
-		(start 140.462 73.66)
-		(end 149.098 73.66)
+		(start 133.767 61.468)
+		(end 136.398 61.468)
 		(width 0.508)
 		(layer "F.Cu")
@@
 	)
 	(segment
-		(start 167.64 62.23)
-		(end 167.64 46.99)
+		(start 140.462 73.66)
+		(end 149.098 73.66)
 		(width 0.508)
 		(layer "F.Cu")
@@
 	)
 	(segment
-		(start 149.098 73.66)
-		(end 149.86 72.898)
+		(start 151.384 68.58)
+		(end 166.116 68.58)
 		(width 0.508)
 		(layer "F.Cu")
@@
 	)
 	(segment
-		(start 166.37 45.72)
-		(end 163 45.72)
+		(start 167.64 67.056)
+		(end 167.64 52.07)
 		(width 0.508)
 		(layer "F.Cu")
@@
 	)
 	(segment
-		(start 139.7 72.898)
-		(end 140.462 73.66)
+		(start 149.86 70.104)
+		(end 151.384 68.58)
 		(width 0.508)
 		(layer "F.Cu")
@@
 	)
 	(segment
-		(start 151.13 66.04)
-		(end 163.83 66.04)
+		(start 167.64 52.07)
+		(end 166.116 50.546)
 		(width 0.508)
 		(layer "F.Cu")
@@
 	)
 	(segment
-		(start 167.64 46.99)
-		(end 166.37 45.72)
+		(start 139.7 72.898)
+		(end 140.462 73.66)
 		(width 0.508)
 		(layer "F.Cu")
@@
 	)
 	(segment
-		(start 149.86 67.31)
-		(end 151.13 66.04)
+		(start 149.098 73.66)
+		(end 149.86 72.898)
 		(width 0.508)
 		(layer "F.Cu")
@@
 		(polygon
 			(pts
-				(xy 158.242 54.864) (xy 157.226 55.88) (xy 145.034 55.88) (xy 145.034 53.086) (xy 146.304 52.07)
-				(xy 146.304 47.752) (xy 146.558 47.498) (xy 146.558 44.958) (xy 148.082 44.958) (xy 149.86 46.736)
-				(xy 149.86 50.292) (xy 151.384 51.816) (xy 158.242 51.816)
+				(xy 150.368 60.198) (xy 146.304 56.134) (xy 144.526 56.134) (xy 144.526 52.832) (xy 146.558 50.8)
+				(xy 146.558 47.752) (xy 146.558 47.498) (xy 146.558 44.958) (xy 148.082 44.958) (xy 149.86 46.736)
+				(xy 149.86 54.102) (xy 151.384 55.626) (xy 160.02 55.626) (xy 160.02 60.198)
 			)
 		)
@@
 		(polygon
 			(pts
-				(xy 159.004 59.436) (xy 145.034 59.436) (xy 144.018 57.658) (xy 141.732 57.658) (xy 139.954 56.134)
-				(xy 143.51 56.134) (xy 143.51 51.562) (xy 143.51 51.308) (xy 143.51 48.26) (xy 146.05 48.26) (xy 146.05 51.562)
-				(xy 144.526 52.832) (xy 144.526 56.134) (xy 159.004 56.134)
+				(xy 160.02 64.516) (xy 148.59 64.516) (xy 141.732 57.658) (xy 139.954 56.134) (xy 143.51 56.134)
+				(xy 143.51 51.562) (xy 143.51 51.308) (xy 143.51 48.26) (xy 146.304 48.26) (xy 146.304 51.054) (xy 144.526 52.832)
+				(xy 144.526 56.134) (xy 146.304 56.134) (xy 150.368 60.198) (xy 160.02 60.198)
 			)
 		)
